Commit message: feat: implement TF2 coordinate frame tree for full stack integration
Three silent frame-name mismatches were preventing the EKF, Nav2 costmap,
and fusion_node from functioning. All three are fixed by aligning URDF link
names with what the rest of the stack expects, removing the need for any
manual StaticTransformBroadcaster nodes.

Changes:

src/description/urdf/asket.urdf.xacro
- Rename root link hull → base_link; update all 7 parent-link references.
  EKF (ekf.yaml: base_link_frame) and Nav2 (nav2_params.yaml: robot_base_frame)
  both require a frame named base_link — hull was never published under that name.
- Rename Lidar → lidar and Lidar_joint → lidar_mount; update all joint
  child/parent refs and the <gazebo reference> plugin attachment.
  lidar_driver stamps every LaserScan with frame_id="lidar"; the URDF link
  must match for TF lookups to resolve.
- Rename joints Lidar_joint_joint → lidar_mount_joint, Lidar_joint_001 → lidar_joint.

src/sensors/sensors/camera_driver.py
- Add frame_id ROS parameter (default "front_camera"). Previously hardcoded
  "camera" matched no URDF link, causing fusion_node's TF lookup to silently
  return None on every call and disabling LiDAR-camera projection entirely.

src/bringup/launch/njord.launch.py
- Pass frame_id: "front_camera" to camera_driver node.
- Pass lidar_frame: "lidar", camera_frame: "front_camera" to fusion_node,
  making frame dependencies explicit and overridable.

.gitignore
- Ignore src/description/*.urdf (generated from xacro at launch time by
  njord.launch.py lines 15-19; not source).
- Ignore frames_*.gv and frames_*.pdf (tf2_tools view_frames output).

Result: robot_state_publisher broadcasts the complete static sensor tree
(base_link → lidar_mount → lidar, front_camera, back_camera, GPS, px4) to
/tf_static on startup. Verified with ros2 run tf2_tools view_frames — all
frames present, correct offsets, no disconnected subtrees.

README.md / TODOS.md updated to reflect verified frame tree and completed items.

Co-Authored-By: Claude Sonnet 4.6 <noreply@anthropic.com>

File: src/description/urdf/asket.urdf.xacro (robot description, xacro)
@@ -68,5 +68,5 @@
     </collision>
   </link>
-  <link name="Lidar">
+  <link name="lidar">
     <inertial>
       <mass value="0.05" />
@@ -84,5 +84,5 @@
     </collision>
   </link>
-  <link name="Lidar_joint">
+  <link name="lidar_mount">
     <inertial>
       <mass value="0.015" />
@@ -132,5 +132,5 @@
     </collision>
   </link>
-  <link name="hull">
+  <link name="base_link">
     <inertial>
       <mass value="14" />
@@ -205,5 +205,5 @@
   <joint name="GPS_joint" type="fixed">
     <origin xyz="-0.18827 0 0.174775" rpy="0 0 0" />
-    <parent link="hull" />
+    <parent link="base_link" />
     <child link="GPS" />
   </joint>
@@ -217,29 +217,29 @@
   <joint name="L_prop_body_joint" type="fixed">
     <origin xyz="-0.65 0.28 -0.1" rpy="0 0 0" />
-    <parent link="hull" />
+    <parent link="base_link" />
     <child link="L_prop_body" />
   </joint>
-  <joint name="Lidar_joint_001" type="fixed">
+  <joint name="lidar_joint" type="fixed">
     <origin xyz="0 0 0.0375" rpy="0 0 0" />
-    <parent link="Lidar_joint" />
-    <child link="Lidar" />
-  </joint>
-  <joint name="Lidar_joint_joint" type="fixed">
+    <parent link="lidar_mount" />
+    <child link="lidar" />
+  </joint>
+  <joint name="lidar_mount_joint" type="fixed">
     <origin xyz="-0.103585 0 0.137275" rpy="0 0 -1.570796" />
-    <parent link="hull" />
-    <child link="Lidar_joint" />
+    <parent link="base_link" />
+    <child link="lidar_mount" />
   </joint>
   <joint name="back_camera_joint" type="fixed">
     <origin xyz="-0.62 -0.02 0.137275" rpy="0 1.570796 0" />
-    <parent link="hull" />
+    <parent link="base_link" />
     <child link="back_camera" />
   </joint>
   <joint name="front_camera_joint" type="fixed">
     <origin xyz="0 0.02 0.137275" rpy="0 1.570796 0" />
-    <parent link="hull" />
+    <parent link="base_link" />
     <child link="front_camera" />
   </joint>
   <joint name="px4_joint" type="fixed">
-    <parent link="hull" />
+    <parent link="base_link" />
     <child link="px4" />
   </joint>
@@ -253,5 +253,5 @@
   <joint name="r_prop_body_joint" type="fixed">
     <origin xyz="-0.65 -0.28 -0.1" rpy="0 0 0" />
-    <parent link="hull" />
+    <parent link="base_link" />
     <child link="r_prop_body" />
   </joint>
@@ -317,5 +317,5 @@
     </sensor>
   </gazebo>
-  <gazebo reference="Lidar">
+  <gazebo reference="lidar">
     <sensor name="Lidar_sensor" type="gpu_lidar">
       <always_on>true</always_on>

Commit message: feat: integrate PID control loop into Gazebo simulation
Full closed-loop PID control now works in sim (use_sim:=true).

Control chain: /cmd_vel → nav_to_pid → pid_controller → actuator_driver
               → /cmd_vel_gz → bridge → /model/asket/cmd_vel → boat moves

Changes:
- gz_bridge.yaml: bridge to /model/asket/cmd_vel (model-scoped topic that
  VelocityControl actually subscribes to, not global /cmd_vel)
- njord.launch.py: resolve package:// mesh URIs to file:// at launch time;
  add GPS sensor static TF to fix navsat_transform warnings; lazy-import
  nav2_common so launch works without nav2 installed; load pid_gains.yaml
- pid_controller.py: use /imu_driver/imu_raw and /odometry/filtered instead
  of MAVROS topics that don't exist in sim; add nav_msgs import
- actuator_driver.py: add use_sim param — sim path scales effort to m/s and
  publishes /cmd_vel_gz; lazy-import mavros_msgs; add effort deadband to
  prevent IMU noise from drifting the boat at idle
- ekf.yaml: enable velocity from odom0 so EKF exports speed in
  /odometry/filtered during simulation
- pid_gains.yaml: tune ki_speed 0.1 → 0.02 (step-response showed integral
  windup from EKF velocity bias at ki=0.1)
- asket.urdf.xacro: use package:// mesh URIs (resolved to file:// in launch)
- basicWorld.sdf: disable shadow casting to fix WSL2 ogre2 render flicker
- package.xml: add nav_msgs exec_depend

Co-Authored-By: Claude Sonnet 4.6 <noreply@anthropic.com>

File: src/description/urdf/asket.urdf.xacro (robot description, xacro)
@@ -41,10 +41,10 @@
     <visual>
       <geometry>
-        <mesh filename="meshes/L_prop_blade_visual.obj" />
-      </geometry>
-    </visual>
-    <collision>
-      <geometry>
-        <mesh filename="meshes/L_prop_blade_collision.stl" />
+        <mesh filename="package://description/meshes/L_prop_blade_visual.obj" />
+      </geometry>
+    </visual>
+    <collision>
+      <geometry>
+        <mesh filename="package://description/meshes/L_prop_blade_collision.stl" />
       </geometry>
     </collision>
@@ -58,5 +58,5 @@
       <origin xyz="0 0 -0.02131" rpy="0 0 0" />
       <geometry>
-        <mesh filename="meshes/L_prop_body_visual.obj" />
+        <mesh filename="package://description/meshes/L_prop_body_visual.obj" />
       </geometry>
     </visual>
@@ -64,5 +64,5 @@
       <origin xyz="0 0 -0.02131" rpy="0 0 0" />
       <geometry>
-        <mesh filename="meshes/L_prop_body_collision.stl" />
+        <mesh filename="package://description/meshes/L_prop_body_collision.stl" />
       </geometry>
     </collision>
@@ -140,5 +140,5 @@
       <origin xyz="0.05313 -0.000017 -0.013484" rpy="0 0 0" />
       <geometry>
-        <mesh filename="meshes/hull_visual.obj" />
+        <mesh filename="package://description/meshes/hull_visual.obj" />
       </geometry>
       <material name="hull" />
@@ -147,5 +147,5 @@
       <origin xyz="0.053118 -0.000017 -0.013613" rpy="0 0 0" />
       <geometry>
-        <mesh filename="meshes/hull_collision.stl" />
+        <mesh filename="package://description/meshes/hull_collision.stl" />
       </geometry>
     </collision>
@@ -175,10 +175,10 @@
     <visual>
       <geometry>
-        <mesh filename="meshes/r_prop_blade_visual.obj" />
-      </geometry>
-    </visual>
-    <collision>
-      <geometry>
-        <mesh filename="meshes/r_prop_blade_collision.stl" />
+        <mesh filename="package://description/meshes/r_prop_blade_visual.obj" />
+      </geometry>
+    </visual>
+    <collision>
+      <geometry>
+        <mesh filename="package://description/meshes/r_prop_blade_collision.stl" />
       </geometry>
     </collision>
@@ -192,5 +192,5 @@
       <origin xyz="0 0 -0.021311" rpy="0 0 0" />
       <geometry>
-        <mesh filename="meshes/r_prop_body_visual.obj" />
+        <mesh filename="package://description/meshes/r_prop_body_visual.obj" />
       </geometry>
     </visual>
@@ -198,5 +198,5 @@
       <origin xyz="0 0 -0.021311" rpy="0 0 0" />
       <geometry>
-        <mesh filename="meshes/r_prop_body_collision.stl" />
+        <mesh filename="package://description/meshes/r_prop_body_collision.stl" />
       </geometry>
     </collision>

Commit message: Fix LiDAR mount yaw sign in URDF (-90deg -> +90deg)
Verified empirically: placed an object measured dead ahead of the
boat and echoed /lidar_driver/scan_raw — it read as lidar-local
(x~=0, y~=-range). Only +90deg predicts that sign; the previous
-90deg predicts the opposite (y~=+range).

This joint feeds base_link<->lidar TF used by anything that consumes
/obstacles/lidar through tf2 (e.g. Nav2's costmap layers) — with the
wrong sign, an obstacle dead ahead of the boat would resolve to
roughly 180 degrees away from its true position in map/base_link
frame. Does not affect the LiDAR-camera calibration tool itself,
which works entirely in the LiDAR's own raw (x,y) consistently
without needing this TF.

Co-Authored-By: Claude Sonnet 5 <noreply@anthropic.com>

File: src/description/urdf/asket.urdf.xacro (robot description, xacro)
@@ -226,5 +226,8 @@
   </joint>
   <joint name="lidar_mount_joint" type="fixed">
-    <origin xyz="-0.103585 0 0.137275" rpy="0 0 -1.570796" />
+    <!-- yaw verified empirically: an object measured dead ahead of the boat
+         reads as lidar-local (x~=0, y~=-range), which only +90deg predicts
+         (the previous -90deg predicted the opposite sign). -->
+    <origin xyz="-0.103585 0 0.137275" rpy="0 0 1.570796" />
     <parent link="base_link" />
     <child link="lidar_mount" />
